File: aquarium.kicad_pcb (KiCad board)
At the start: 2 copper layers, 104 x 47 mm, 40 parts, among them U1 MOC3063, U2 MOC3063

Commit message: New version of the controller (schematic and pcb).
Parts:
- removed G***: LOGO, aquarium:logo
- removed VS2: BT137, Транзисторы:TO220
- added C10: 6.8мк, Конденсаторы:CPH_5_10x16mm, B.Cu at (84.2, 120.5)
- added C11: 22мк, Конденсаторы:CPH_5_13x25mm, B.Cu at (84.2, 108.5)
- added C12: 100н, Конденсаторы:C_5x3mm, B.Cu at (115.8, 110.2)
- added C13: 10н, Конденсаторы:C_7.5x4mm, B.Cu at (85.5, 95.8)
- added C14: 2н2, Конденсаторы:C_7.5x4mm, B.Cu at (108.2, 123.2)
- added C15: 1000мк, Конденсаторы:CPH_5_10x20mm, B.Cu at (113.5, 84.5)
- added C16: 100мк, Конденсаторы:CP_2.5x6mm, B.Cu at (131.5, 101.5)
- added C17: 47мк, Конденсаторы:CP_2.5x5mm, B.Cu at (128.2, 112.5)
- added C9: 0.1, Конденсаторы:SMD_0805, F.Cu at (215.2, 111.7)
- added DA2: 78L05, Транзисторы:TO92-250, B.Cu at (128.2, 107.2)
- added DD5: DS18B20, Разъемы:PLS-3, B.Cu at (150.5, 84.3)
- added FU1: 3.15A, Прочее:FU_5x20mm, B.Cu at (64.0, 114.0)
- added L1: 1мГн, Дроссели:Ind_5x8mm, B.Cu at (72.2, 100.8)
- added L2: 100мкГн, Дроссели:Ind_5x8mm, B.Cu at (130.2, 94.0)
- added R13: 1M8, Резисторы:RV_0.25, B.Cu at (110.5, 117.0)
- added R14: 1к, Резисторы:RV_0.25, B.Cu at (77.5, 94.5)
- added R15: 100, Резисторы:RV_0.25, B.Cu at (92.5, 97.8)
- added R16: 390, Резисторы:RV_0.25, B.Cu at (123.8, 123.2)
- added R17: 2к, Резисторы:RV_0.25, B.Cu at (117.0, 123.2)
- added RU1: 275B, Резисторы:FNR-05, B.Cu at (56.2, 102.5)
- added T1: E16, Трансформаторы:E16_5_10mm, B.Cu at (103.2, 93.2)
- added VD1: 1N4007, Диоды:DO-41, B.Cu at (75.5, 118.0)
- added VD2: 1N4007, Диоды:DO-41, B.Cu at (75.5, 123.0)
- added VD3: 1N4007, Диоды:DO-41, B.Cu at (75.5, 113.0)
- added VD4: 1N4007, Диоды:DO-41, B.Cu at (75.5, 108.0)
- added VD5: P6KE150A, Диоды:DO-15, B.Cu at (84.5, 99.8)
- added VD6: UF4007, Диоды:DO-41, B.Cu at (87.5, 91.0)
- added VD7: 1N5819, Диоды:DO-41, B.Cu at (117.5, 93.2)
- added VD8: 1N4741A, Диоды:DO-41, B.Cu at (129.0, 119.7)
- added VT1: IRLD014, Транзисторы:HVMDIP, B.Cu at (160.6, 120.2)
- added XP2: Sensor 2, Разъемы:PLS-1, B.Cu at (235.7, 86.8)
- added XT7: PLS-4, Разъемы:PLS-4, B.Cu at (132.5, 112.7)
- C2: value 2n2 -> 0.1
- C5, C6: value 0.1 -> 3n3
- DA1: value 78L05 -> TNY274; footprint Транзисторы:TO92-250 -> Микросхемы:PDIP-8C
- DD1: value DS18B20 -> ATMEGA8A; footprint Разъемы:PLS-3 -> Микросхемы:TQFP32-30; moved to F.Cu
- DD3: value DS1302 -> AT42QT1011; footprint Микросхемы:DIP8-300 -> Транзисторы:SOT23-6; moved to F.Cu
- DD4: value ATMEGA8A -> DS1302; footprint Микросхемы:TQFP32-30 -> Микросхемы:DIP8-300; moved to B.Cu
- GB1: value 3V -> 3В
- R1: value 100k -> 30
- R10, R9: value 30 -> 360; footprint Резисторы:R_0805 -> Резисторы:RH_2; moved to B.Cu
- R11: value 30 -> 620; footprint Резисторы:R_0805 -> Резисторы:RV_0.25; moved to B.Cu
- R12: value 30 -> 1M8; footprint Резисторы:R_0805 -> Резисторы:RV_0.25; moved to B.Cu
- R2, R3, R4, R5: value 360 -> 30; footprint Резисторы:RH_2 -> Резисторы:R_0805; moved to F.Cu
- R7, R8: value 620 -> 100k
- U2: value MOC3063 -> PC817A; footprint Микросхемы:DIP6-300 -> Микросхемы:DIP4-300
- XP1: value Sensor -> Sensor 1
- XT1, XT3: value DG350-3.5-02P-14 -> PLS-4; footprint Разъемы:DG-350-2 -> Разъемы:PLS-4
- XT2: value DG350-3.5-02P-14 -> PLS-6; footprint Разъемы:DG-350-2 -> Разъемы:PLS-6
- XT5: value PLS-4 -> DG350-3.5-02P-14; footprint Разъемы:PLS-4 -> Разъемы:DG-350-2
- XT6: value PLD-6 -> DG350-3.5-02P-14; footprint Разъемы:PLD-6 -> Разъемы:DG-350-2
- ZQ1: footprint Резисторы:R_0805 -> Прочее:HC_3.0x8.0mm; moved to B.Cu
- moved XP1 142.1 mm to (235.8, 97.0), turned to 0 degrees
- moved C2 124.7 mm to (220.5, 86.8)
- moved DD2 122.0 mm to (224.2, 97.0), turned to 0 degrees
- moved VS1 120.5 mm to (65.7, 92.8), turned to 0 degrees
- moved C6 118.9 mm to (228.0, 86.8), turned to 270 degrees
- moved C7 118.0 mm to (212.2, 95.2), turned to 270 degrees
- moved C5 114.9 mm to (228.1, 97.0), turned to 270 degrees
- moved DD1 109.5 mm to (205.2, 94.1), turned to 0 degrees
- moved XT2 104.5 mm to (198.1, 111.2), turned to 45 degrees
- moved XT6 101.7 mm to (56.2, 84.8), turned to 90 degrees
- moved DD3 99.4 mm to (224.2, 86.8), turned to 0 degrees
- moved C4 95.5 mm to (197.2, 94.0), turned to 270 degrees
- moved DD4 95.2 mm to (207.1, 112.8), turned to 225 degrees
- moved C1 93.5 mm to (220.5, 97.0), turned to 90 degrees
- moved U1 89.1 mm to (89.8, 84.8), turned to 270 degrees
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Connections:
- C1 pad 1: +5B -> /SENS_PWR
- C2 pad 1: Net-(C2-Pad1) -> /SENS_PWR
- C2 pad 2: Net-(C2-Pad2) -> GND
- C3 pad 1: +5B -> /TEMP_PWR
- C4 pad 1: /~RESET -> +5B
- C5 pad 1: +5B -> Net-(C5-Pad1)
- C5 pad 2: GND -> Net-(C5-Pad2)
- C6 pad 1: +5B -> Net-(C6-Pad1)
- C6 pad 2: GND -> Net-(C6-Pad2)
- C7 pad 1: Vin -> +5B
- C8 pad 1: +5B -> /~RESET
- DA1 pad 1: +5B -> Net-(DA1-Pad1)
- DA1 pad 2: GND -> Net-(C12-Pad1)
- DD1 pad 1: GND -> /F
- DD1 pad 2: /TEMP -> /A
- DD1 pad 3: +5B -> GND
- DD2 pad 1: /SENS -> /SENS_1
- DD2 pad 3: Net-(C2-Pad1) -> Net-(C5-Pad1)
- DD2 pad 4: Net-(C2-Pad2) -> Net-(C5-Pad2)
- DD2 pad 5: +5B -> /SENS_PWR
- DD2 pad 6: +5B -> /SENS_PWR
- DD3 pad 1: +5B -> /SENS_2
- DD3 pad 2: Net-(DD3-Pad2) -> GND
- DD3 pad 3: Net-(DD3-Pad3) -> Net-(C6-Pad1)
- DD3 pad 4: GND -> Net-(C6-Pad2)
- DD3 pad 5: /RTC_CE -> /SENS_PWR
- DD3 pad 6: /RTC_IO -> /SENS_PWR
- DD4 pad 1: /TEMP -> +5B
- DD4 pad 2: /SENS -> Net-(DD4-Pad2)
- DD4 pad 3: GND -> Net-(DD4-Pad3)
- DD4 pad 4: +5B -> GND
- DD4 pad 5: GND -> /MISO
- DD4 pad 6: +5B -> /RTC_IO
- DD4 pad 7: /RTC_SCLK -> /MOSI
- DD4 pad 8: /RTC_IO -> Net-(DD4-Pad8)
- GB1 pad 1: VBAT -> Net-(DD4-Pad8)
- R1 pad 1: Net-(R1-Pad1) -> /DGT4
- R1 pad 2: Net-(C2-Pad1) -> Net-(HG1-Pad6)
- R10 pad 1: /DGT2 -> Net-(R10-Pad1)
- R10 pad 2: Net-(HG1-Pad9) -> Net-(R10-Pad2)
- R11 pad 1: /DGT3 -> Net-(R11-Pad1)
- R11 pad 2: Net-(HG1-Pad8) -> Net-(R11-Pad2)
- R12 pad 1: /DGT4 -> Net-(C10-Pad1)
- R12 pad 2: Net-(HG1-Pad6) -> Net-(R12-Pad2)
- R2 pad 1: Net-(R2-Pad1) -> /DGT3
- R2 pad 2: Net-(R2-Pad2) -> Net-(HG1-Pad8)
- R3 pad 1: Net-(R3-Pad1) -> /DGT2
- R3 pad 2: Net-(R3-Pad2) -> Net-(HG1-Pad9)
- R4 pad 1: Net-(R4-Pad1) -> /LIGHT
- R4 pad 2: Net-(R2-Pad2) -> Net-(R4-Pad2)
- R5 pad 1: Net-(R5-Pad1) -> /DGT1
- R5 pad 2: Net-(R5-Pad2) -> Net-(HG1-Pad12)
- R6 pad 1: +5B -> /TEMP
- R6 pad 2: /TEMP -> /TEMP_PWR
- R7 pad 2: /HEAT -> Net-(C5-Pad1)
- R8 pad 2: /LIGHT -> Net-(C6-Pad1)
- R9 pad 1: /DGT1 -> Net-(R9-Pad1)
- R9 pad 2: Net-(HG1-Pad12) -> Net-(FU1-Pad2)
- U1 pad 1: Net-(R7-Pad1) -> Net-(R11-Pad1)
- U1 pad 4: Net-(R3-Pad1) -> Net-(R10-Pad1)
- U1 pad 6: Net-(R2-Pad1) -> Net-(R9-Pad1)
- U2 pad 1: Net-(R8-Pad1) -> Net-(R16-Pad2)
- U2 pad 3: (no net) -> Net-(C11-Pad2)
- U2 pad 4: Net-(R5-Pad1) -> Net-(DA1-Pad1)
- VS1 pad 1: Net-(R3-Pad2) -> Net-(R10-Pad2)
- VS1 pad 2: Net-(R2-Pad2) -> Net-(FU1-Pad2)
- VS1 pad 3: Net-(R3-Pad1) -> Net-(R10-Pad1)
- XP1 pad 1: Net-(R1-Pad1) -> Net-(R7-Pad1)
- XT1 pad 1: Vin -> +5B
- XT2 pad 1: Net-(R2-Pad2) -> /~RESET
- XT2 pad 2: Net-(XT2-Pad2) -> +5B
- XT3 pad 1: Net-(R3-Pad2) -> +12B
- XT3 pad 2: Net-(XT2-Pad2) -> +5B
- XT4 pad 1: Net-(R5-Pad2) -> +12B
- XT4 pad 2: Net-(XT2-Pad2) -> Net-(VT1-Pad1)
- XT5 pad 1: +5B -> Net-(FU1-Pad1)
- XT5 pad 2: /TX -> Net-(RU1-Pad1)
- XT6 pad 1: /E -> Net-(RU1-Pad1)
- XT6 pad 2: +5B -> Net-(R10-Pad2)
- ZQ1 pad 1: Net-(DD3-Pad3) -> Net-(DD4-Pad3)
- ZQ1 pad 2: Net-(DD3-Pad2) -> Net-(DD4-Pad2)
Routing:
- net Net-(R2-Pad2): track 153.4 -> 0.00 mm
- net GND: track 246.7 -> 395.8 mm, vias 0 -> 4
- net Net-(XT2-Pad2): track 126.9 -> 0.00 mm
- net +5B: track 83.9 -> 169.0 mm
- net /TEMP_PWR: track 0.00 -> 71.2 mm
- net /RX: track 17.8 -> 86.8 mm, vias 0 -> 2
- net Net-(C11-Pad2): track 0.00 -> 66.7 mm
- net Net-(C10-Pad1): track 0.00 -> 62.5 mm
- net Net-(RU1-Pad1): track 0.00 -> 62.3 mm
- net Net-(R11-Pad2): track 0.00 -> 60.2 mm
- net Net-(C15-Pad1): track 0.00 -> 55.6 mm, vias 0 -> 2
- net Net-(FU1-Pad2): track 0.00 -> 49.1 mm
- net /TX: track 16.5 -> 62.5 mm, vias 0 -> 2
- net /TEMP: track 18.6 -> 64.4 mm
- net +12B: track 0.00 -> 40.4 mm, vias 0 -> 2
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- removed copper zone on F.Cu, net +5B
Other:
- board size 104 x 47 mm -> 190.8 x 47 mm
- net class Default: trace_width 0.25 -> 0.4; via_dia 0.6 -> 2; via_drill 0.4 -> 0.8
- board text added: "+"
- board text added: "+12V"
- board text added: "-"
- board text added: "MISO"
- board text added: "MOSI"
- board text added: "PICkit2"
- board text added: "SCK"
- board text added: "VCC"
- board text added: "~RESET"
- board text removed: "1"
- board text removed: "ISP"

Commit message: Small changes to PCB.
Parts:
- C13: footprint Конденсаторы:C_7.5x4mm -> Конденсаторы:C_5x3mm
- moved C13 0.50 mm to (85.0, 95.8)
Routing:
- net Net-(C13-Pad1): track 3.25 -> 5.00 mm
- net Net-(C13-Pad2): track 10.7 -> 9.75 mm
Changed lines of the file:
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@@
-(kicad_pcb (version 20160815) (host pcbnew "(2016-12-30 revision d5ce0a8ee)-new_icons")
+(kicad_pcb (version 20160815) (host pcbnew "(2017-01-18 revision 02e05552a)-new_icons")
   (general
     (links 155)
-    (no_connects 3)
+    (no_connects 5)
     (area 49.424999 78.924999 240.325001 126.075001)
     (thickness 1.6)
     (drawings 40)
-    (tracks 524)
+    (tracks 523)
     (zones 0)
     (modules 70)
@@
   )
   (setup
-    (last_trace_width 1)
+    (last_trace_width 1.5)
     (user_trace_width 0.2)
     (user_trace_width 0.3)
@@
     (mod_text_size 1 1)
     (mod_text_width 0.15)
-    (pad_size 2.5 2.5)
+    (pad_size 2.6 2.6)
     (pad_drill 0.8)
     (pad_to_mask_clearance 0.2)
@@
     (add_net "Net-(VT1-Pad1)")
   )
+  (module Конденсаторы:C_5x3mm (layer B.Cu)
+    (at 85 95.75 180)
+    (fp_text reference C13 (at 2.25 2.25 180) (layer B.SilkS)
+      (effects (font (size 1 1) (thickness 0.15)) (justify mirror))
+    )
+    (fp_text value 10н (at 0 0 180) (layer B.SilkS)
+      (effects (font (size 1 1) (thickness 0.15)) (justify mirror))
+    )
+    (fp_arc (start 0 6) (end 3.5 -0.5) (angle -56.6) (layer B.SilkS) (width 0.254))
+    (fp_arc (start 0 -6) (end -3.5 0.5) (angle -56.6) (layer B.SilkS) (width 0.254))
+    (fp_line (start -3.5 0.5) (end -3.5 -0.5) (layer B.SilkS) (width 0.254))
+    (fp_line (start 3.5 0.5) (end 3.5 -0.5) (layer B.SilkS) (width 0.254))
+    (pad 1 thru_hole circle (at -2.5 0 180) (size 2.6 2.6) (drill 0.8) (layers *.Cu *.Mask B.SilkS)
+      (net 37 "Net-(C13-Pad1)"))
+    (pad 2 thru_hole circle (at 2.5 0 180) (size 2.6 2.6) (drill 0.8) (layers *.Cu *.Mask B.SilkS)
+      (net 38 "Net-(C13-Pad2)"))
+  )
   (module Трансформаторы:E16_5_10mm (layer B.Cu)
     (at 103.25 93.25 270)
     (descr "Импульсный траныформатор E16")
-    (fp_text reference T1 (at -9.25 -6.5 360) (layer B.SilkS)
+    (fp_text reference T1 (at -9.25 -6.5) (layer B.SilkS)
       (effects (font (size 1 1) (thickness 0.15)) (justify mirror))
     )
@@
     (descr "4 pins DIL package, round pads")
     (tags DIL)
-    (fp_text reference VT1 (at 3.81 0 360) (layer B.SilkS)
-      (effects (font (size 1 1) (thickness 0.15)) (justify mirror))
-    )
-    (fp_text value IRLD014 (at 0 -0.06 360) (layer B.SilkS) hide
+    (fp_text reference VT1 (at 3.81 0) (layer B.SilkS)
+      (effects (font (size 1 1) (thickness 0.15)) (justify mirror))
+    )
+    (fp_text value IRLD014 (at 0 -0.06) (layer B.SilkS) hide
       (effects (font (size 1 1) (thickness 0.15)) (justify mirror))
     )
@@
     (descr "Capacitor smd 0805")
     (tags C)
-    (fp_text reference C5 (at -3.25 0 360) (layer F.SilkS)
+    (fp_text reference C5 (at -3.25 0) (layer F.SilkS)
       (effects (font (size 1 1) (thickness 0.15)))
     )
@@
     (descr "Capacitor smd 0805")
     (tags C)
-    (fp_text reference C6 (at -3.175 0 360) (layer F.SilkS)
+    (fp_text reference C6 (at -3.175 0) (layer F.SilkS)
       (effects (font (size 1 1) (thickness 0.15)))
     )
@@
   (module Разъемы:CR2032_H (layer B.Cu)
     (at 225.495 111.57 315)
-    (fp_text reference GB1 (at -13.834544 -0.053033 585) (layer B.SilkS)
-      (effects (font (size 1 1) (thickness 0.15)) (justify mirror))
-    )
-    (fp_text value 3В (at 3 0 405) (layer B.SilkS)
+    (fp_text reference GB1 (at -13.834544 -0.053033 225) (layer B.SilkS)
+      (effects (font (size 1 1) (thickness 0.15)) (justify mirror))
+    )
+    (fp_text value 3В (at 3 0 45) (layer B.SilkS)
       (effects (font (size 1 1) (thickness 0.15)) (justify mirror))
     )
@@
     (descr "6 pins DIL package, round pads")
     (tags DIL)
-    (fp_text reference U1 (at -5 0 360) (layer B.SilkS)
+    (fp_text reference U1 (at -5 0) (layer B.SilkS)
       (effects (font (size 1 1) (thickness 0.15)) (justify mirror))
     )
@@
   (module Разъемы:DG-350-2 (layer B.Cu)
     (at 150.5 119.73 270)
-    (fp_text reference XT4 (at -4.75 0 360) (layer B.SilkS)
+    (fp_text reference XT4 (at -4.75 0) (layer B.SilkS)
       (effects (font (size 1 1) (thickness 0.15)) (justify mirror))
     )
@@
     (descr "Resistor smd 0805")
     (tags "R RES")
-    (fp_text reference R6 (at 2.81 0 360) (layer F.SilkS)
+    (fp_text reference R6 (at 2.81 0) (layer F.SilkS)
       (effects (font (size 1 1) (thickness 0.15)))
     )
@@
   )
   (module Конденсаторы:C_7.5x4mm (layer B.Cu)
-    (at 85.5 95.75 180)
-    (fp_text reference C13 (at -5.5 2 180) (layer B.SilkS)
-      (effects (font (size 1 1) (thickness 0.15)) (justify mirror))
-    )
-    (fp_text value 10н (at 0 0 180) (layer B.SilkS) hide
-      (effects (font (size 1 1) (thickness 0.15)) (justify mirror))
-    )
-    (fp_arc (start 0 -8) (end -5 0.75) (angle -59.4) (layer B.SilkS) (width 0.254))
-    (fp_line (start 5 0.75) (end 5 -0.75) (layer B.SilkS) (width 0.254))
-    (fp_line (start -5 -0.75) (end -5 0.75) (layer B.SilkS) (width 0.254))
-    (fp_arc (start 0 8) (end 5 -0.75) (angle -59.4) (layer B.SilkS) (width 0.254))
-    (pad 1 thru_hole circle (at -3.75 0 180) (size 2.6 2.6) (drill 0.8) (layers *.Cu *.Mask B.SilkS)
-      (net 37 "Net-(C13-Pad1)"))
-    (pad 2 thru_hole circle (at 3.75 0 180) (size 2.6 2.6) (drill 0.8) (layers *.Cu *.Mask B.SilkS)
-      (net 38 "Net-(C13-Pad2)"))
-  )
-  (module Конденсаторы:C_7.5x4mm (layer B.Cu)
     (at 108.25 123.25 180)
-    (fp_text reference C14 (at -4 2.5 360) (layer B.SilkS)
+    (fp_text reference C14 (at -4 2.5) (layer B.SilkS)
       (effects (font (size 1 1) (thickness 0.15)) (justify mirror))
     )
@@
     (at 128.25 112.5 45)
     (descr "Capacitor, pol, cyl 6x11mm")
-    (fp_text reference C17 (at -2.487436 2.65165 360) (layer B.SilkS)
+    (fp_text reference C17 (at -2.487436 2.65165) (layer B.SilkS)
       (effects (font (size 1 1) (thickness 0.15)) (justify mirror))
     )
@@
     (fp_circle (center 0 0) (end 0 -2.5) (layer B.SilkS) (width 0.254))
     (fp_line (start -1.25 1.75) (end -1.25 0.75) (layer B.SilkS) (width 0.254))
-    (pad 1 thru_hole rect (at -1.25 0 45) (size 1.6 1.6) (drill 0.8) (layers *.Cu *.Mask B.SilkS)
+    (pad 1 thru_hole rect (at -1.249999 0 45) (size 1.6 1.6) (drill 0.8) (layers *.Cu *.Mask B.SilkS)
       (net 2 +5B))
-    (pad 2 thru_hole circle (at 1.25 0 45) (size 1.6 1.6) (drill 0.8) (layers *.Cu *.Mask B.SilkS)
+    (pad 2 thru_hole circle (at 1.249999 0 45) (size 1.6 1.6) (drill 0.8) (layers *.Cu *.Mask B.SilkS)
       (net 1 GND))
   )
@@
     (descr "DIL package, round pads")
     (tags DIL)
-    (fp_text reference DA1 (at -0.06 6.06 360) (layer B.SilkS)
+    (fp_text reference DA1 (at -0.06 6.06) (layer B.SilkS)
       (effects (font (size 1 1) (thickness 0.15)) (justify mirror))
     )
@@
   (module Резисторы:RV_0.25 (layer B.Cu)
     (at 77.5 94.5 270)
-    (fp_text reference R14 (at -2 3.5 360) (layer B.SilkS)
+    (fp_text reference R14 (at -2 3.5) (layer B.SilkS)
       (effects (font (size 1 1) (thickness 0.15)) (justify mirror))
     )
@@
   (module Диоды:DO-41 (layer B.Cu)
     (at 87.5 91 180)
-    (fp_text reference VD6 (at 6.25 -2.25 180) (layer B.SilkS)
+    (fp_text reference VD6 (at 0 -2.5 180) (layer B.SilkS)
       (effects (font (size 1 1) (thickness 0.15)) (justify mirror))
     )
@@
   (segment (start 118.25 110.25) (end 118.25 107.41) (width 1.5) (layer F.Cu) (net 36))
   (segment (start 118.25 107.41) (end 118.21 107.37) (width 1.5) (layer F.Cu) (net 36))
-  (segment (start 89.25 95.75) (end 92.5 95.75) (width 1.5) (layer F.Cu) (net 37))
-  (segment (start 77.5 92.5) (end 81 92.5) (width 1.5) (layer F.Cu) (net 38))
-  (segment (start 81 92.5) (end 82.5 91) (width 1.5) (layer F.Cu) (net 38))
-  (segment (start 81.75 95.75) (end 81.75 91.75) (width 1.5) (layer F.Cu) (net 38))
-  (segment (start 81.75 91.75) (end 82.5 91) (width 1.5) (layer F.Cu) (net 38))
+  (segment (start 87.5 95.75) (end 92.5 95.75) (width 1.5) (layer F.Cu) (net 37))
+  (segment (start 82.5 95.75) (end 82.5 92.5) (width 1.5) (layer F.Cu) (net 38))
+  (segment (start 82.5 92.5) (end 82.5 91) (width 1.5) (layer F.Cu) (net 38))
+  (segment (start 77.5 92.5) (end 82.5 92.5) (width 1.5) (layer F.Cu) (net 38))
   (segment (start 124 117.5) (end 124 116.085787) (width 0.4) (layer B.Cu) (net 39))
   (segment (start 124 116.085787) (end 124 95.25) (width 0.4) (layer B.Cu) (net 39))

Commit message: Finished working on PCB.
Parts:
- added G***: LOGO, aquarium:oshw-logo, B.Cu at (28.8, 75.2)
- added REF**: Symbol_HighVoltage_Type2_CopperTop_VerySmall, Symbols:Symbol_HighVoltage_Type2_CopperTop_VerySmall, B.Cu at (55.8, 7.50)
- R11: footprint Резисторы:RV_0.25 -> Резисторы:RH_0.25
- moved C1 142.0 mm to (80.8, 72.0)
- moved C2 142.0 mm to (80.8, 61.8)
- moved C3 142.0 mm to (7.50, 59.2)
- moved C4 142.0 mm to (57.5, 69.0)
- moved C5 142.0 mm to (88.3, 72.0)
- moved C6 142.0 mm to (88.2, 61.8)
- moved C7 142.0 mm to (72.5, 70.2)
- moved C8 142.0 mm to (51.0, 92.0)
- moved C9 142.0 mm to (75.5, 86.7)
- moved DD1 142.0 mm to (65.4, 69.1)
- moved DD2 142.0 mm to (84.5, 72.0)
- moved DD3 142.0 mm to (84.5, 61.8)
- moved DD4 142.0 mm to (67.3, 87.8)
- moved DD5 142.0 mm to (10.8, 59.3)
- moved GB1 142.0 mm to (85.7, 86.6)
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Routing:
- net Net-(R11-Pad2): track 60.2 -> 2.25 mm
- net Net-(C15-Pad1): track 55.6 -> 24.6 mm, vias 2 -> 0
- net Net-(R9-Pad1): track 2.03 -> 31.6 mm
- net Net-(R10-Pad1): track 20.0 -> 47.6 mm
- net Net-(C10-Pad1): track 62.5 -> 84.4 mm
- net Net-(C11-Pad2): track 66.7 -> 47.6 mm
- net +12B: track 40.4 -> 21.8 mm, vias 2 -> 0
- net +5B: track 169.0 -> 186.9 mm
- net Net-(DA1-Pad4): track 27.4 -> 11.5 mm
- net GND: track 395.8 -> 381.3 mm
- net Net-(C10-Pad2): track 33.8 -> 21.2 mm
- net Net-(C12-Pad1): track 2.90 -> 14.9 mm
- net Net-(T1-Pad3): track 2.75 -> 8.41 mm
- net Net-(DA1-Pad1): track 15.6 -> 20.8 mm
- net Net-(R16-Pad2): track 5.74 -> 10.1 mm
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Other:
- board size 190.8 x 47 mm -> 96.2 x 98 mm
- board text added: "SENSOR 1"
- board text added: "SENSOR 2"

Commit message: New version of the schematic and PCB's.
Parts:
- added R18: 470, Резисторы:R_0805, F.Cu at (62.4, 84.8)
Connections:
- DD4 pad 6: /RTC_IO -> Net-(DD4-Pad6)
Routing:
- net /RTC_IO: track 23.0 -> 19.2 mm
Changed lines of the file:
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@@
-(kicad_pcb (version 20170123) (host pcbnew "(2017-01-31 revision 5d64ff7e8)-new_icons")
+(kicad_pcb (version 20170123) (host pcbnew "(2017-02-20 revision 5c7030387)-new_icons_rebased")
   (general
-    (links 0)
+    (links 156)
     (no_connects 6)
-    (area 3.924999 2.924999 100.325001 101.075001)
+    (area 3.902999 0.594047 100.325001 102.885952)
     (thickness 1.6)
     (drawings 47)
-    (tracks 520)
+    (tracks 519)
     (zones 0)
-    (modules 72)
-    (nets 66)
+    (modules 73)
+    (nets 67)
   )
   (page User 105.004 105.004)
@@
     (visible_elements FFFFFFFF)
     (pcbplotparams
-      (layerselection 0x00010_7ffffffe)
+      (layerselection 0x00030_7fffffff)
       (usegerberextensions false)
       (excludeedgelayer false)
@@
   (net 64 "Net-(VT1-Pad1)")
   (net 65 "Net-(R14-Pad2)")
+  (net 66 "Net-(DD4-Pad6)")
   (net_class Default "This is the default net class."
     (clearance 0.2)
@@
     (add_net "Net-(DD4-Pad2)")
     (add_net "Net-(DD4-Pad3)")
+    (add_net "Net-(DD4-Pad6)")
     (add_net "Net-(DD4-Pad8)")
     (add_net "Net-(FU1-Pad1)")
@@
       (net 44 /MISO))
     (pad 6 thru_hole oval (at 1.27 3.81 225) (size 1.5 3) (drill 0.8) (layers *.Cu *.Mask B.SilkS)
-      (net 10 /RTC_IO))
+      (net 66 "Net-(DD4-Pad6)"))
     (pad 7 thru_hole oval (at -1.27 3.81 225) (size 1.5 3) (drill 0.8) (layers *.Cu *.Mask B.SilkS)
       (net 43 /MOSI))
@@
       (net 58 "Net-(R11-Pad2)"))
   )
+  (module Резисторы:R_0805 (layer F.Cu)
+    (at 62.4 84.8 315)
+    (descr "Resistor smd 0805")
+    (tags "R RES")
+    (fp_text reference R18 (at -4.666905 0 315) (layer F.SilkS)
+      (effects (font (size 1 1) (thickness 0.15)))
+    )
+    (fp_text value 470 (at 0.1 0 315) (layer F.SilkS) hide
+      (effects (font (size 1 1) (thickness 0.15)))
+    )
+    (fp_line (start 0.762 -1.016) (end 1.905 -1.016) (layer F.SilkS) (width 0.254))
+    (fp_line (start 1.905 -1.016) (end 1.905 1.016) (layer F.SilkS) (width 0.254))
+    (fp_line (start 1.905 1.016) (end 0.762 1.016) (layer F.SilkS) (width 0.254))
+    (fp_line (start -1.905 -1.016) (end -0.762 -1.016) (layer F.SilkS) (width 0.254))
+    (fp_line (start -1.905 1.016) (end -1.905 -1.016) (layer F.SilkS) (width 0.254))
+    (fp_line (start -1.905 1.016) (end -0.762 1.016) (layer F.SilkS) (width 0.254))
+    (pad 1 smd rect (at 1 0 315) (size 1.3 1.5) (layers F.Cu)
+      (net 66 "Net-(DD4-Pad6)"))
+    (pad 2 smd rect (at -1 0 315) (size 1.3 1.5) (layers F.Cu)
+      (net 10 /RTC_IO))
+  )
   (gr_text "SENSOR 2" (at 94 61.7) (layer B.SilkS)
     (effects (font (size 1 1) (thickness 0.15)) (justify left mirror))
@@
   (gr_circle (center 51.75 92.75) (end 51.75 93) (layer B.SilkS) (width 0.3))
   (gr_circle (center 51.75 92.75) (end 52.25 92.75) (layer B.SilkS) (width 0.2))
-  (gr_text HEAT (at 96.75 7.25) (layer B.SilkS)
+  (gr_text HEAT (at 96.75 6) (layer B.SilkS)
     (effects (font (size 1 1) (thickness 0.15)) (justify mirror))
   )
-  (gr_text +12V (at 97 14.75) (layer B.SilkS)
+  (gr_text +12V (at 97 13.5) (layer B.SilkS)
     (effects (font (size 1 1) (thickness 0.15)) (justify mirror))
   )
-  (gr_text +5V (at 96.5 12.25) (layer B.SilkS)
+  (gr_text +5V (at 96.5 11) (layer B.SilkS)
     (effects (font (size 1 1) (thickness 0.15)) (justify mirror))
   )
-  (gr_text GND (at 96.5 9.75) (layer B.SilkS)
+  (gr_text GND (at 96.5 8.5) (layer B.SilkS)
     (effects (font (size 1 1) (thickness 0.15)) (justify mirror))
   )
@@
     (effects (font (size 2 2) (thickness 0.254)) (justify mirror))
   )
-  (gr_text +12V (at 6.75 87.75) (layer B.SilkS)
+  (gr_text +12V (at 6.75 86.5) (layer B.SilkS)
     (effects (font (size 1 1) (thickness 0.15)) (justify mirror))
   )
-  (gr_text HEAT (at 7 80.25) (layer B.SilkS)
+  (gr_text HEAT (at 7 79) (layer B.SilkS)
     (effects (font (size 1 1) (thickness 0.15)) (justify mirror))
   )
-  (gr_text GND (at 7.37 63) (layer B.SilkS)
+  (gr_text GND (at 7.37 62) (layer B.SilkS)
     (effects (font (size 1 1) (thickness 0.15)) (justify mirror))
   )
-  (gr_text DQ (at 7.75 60.5) (layer B.SilkS)
+  (gr_text DQ (at 7.75 59.5) (layer B.SilkS)
     (effects (font (size 1 1) (thickness 0.15)) (justify mirror))
   )
-  (gr_text VDD (at 7.37 57.97) (layer B.SilkS)
+  (gr_text VDD (at 7.37 56.97) (layer B.SilkS)
     (effects (font (size 1 1) (thickness 0.15)) (justify mirror))
   )
@@
     (effects (font (size 1 1) (thickness 0.15)) (justify mirror))
   )
-  (gr_text GND (at 7.25 82.75) (layer B.SilkS)
+  (gr_text GND (at 7.25 81.5) (layer B.SilkS)
     (effects (font (size 1 1) (thickness 0.15)) (justify mirror))
   )
-  (gr_text +5V (at 7.25 85.25) (layer B.SilkS)
+  (gr_text +5V (at 7.25 84) (layer B.SilkS)
     (effects (font (size 1 1) (thickness 0.15)) (justify mirror))
   )
@@
     (effects (font (size 1 1) (thickness 0.15)) (justify mirror))
   )
-  (gr_text GND (at 7.25 70.5) (layer B.SilkS)
+  (gr_text GND (at 7.5 69.25) (layer B.SilkS)
     (effects (font (size 1 1) (thickness 0.15)) (justify mirror))
   )
-  (gr_text RX (at 7.75 73) (layer B.SilkS)
+  (gr_text RX (at 8 71.75) (layer B.SilkS)
     (effects (font (size 1 1) (thickness 0.15)) (justify mirror))
   )
-  (gr_text TX (at 7.75 75.5) (layer B.SilkS)
+  (gr_text TX (at 8 74.25) (layer B.SilkS)
     (effects (font (size 1 1) (thickness 0.15)) (justify mirror))
   )
-  (gr_text +5V (at 7.25 68) (layer B.SilkS)
+  (gr_text +5V (at 7.5 66.75) (layer B.SilkS)
     (effects (font (size 1 1) (thickness 0.15)) (justify mirror))
   )
@@
   (segment (start 59.86863 81.13137) (end 59.86863 82.36863) (width 0.4) (layer F.Cu) (net 10))
   (segment (start 59.86863 82.36863) (end 61 83.5) (width 0.4) (layer F.Cu) (net 10))
-  (segment (start 63.737898 86.043949) (end 63.543949 86.043949) (width 0.5) (layer F.Cu) (net 10))
-  (segment (start 63.543949 86.043949) (end 61 83.5) (width 0.5) (layer F.Cu) (net 10))
   (segment (start 65.048675 64.833467) (end 65.048675 62.798675) (width 0.4) (layer F.Cu) (net 11))
   (segment (start 65.048675 62.798675) (end 63 60.75) (width 0.4) (layer F.Cu) (net 11))
@@
   (segment (start 16.96 96.48) (end 17 96.52) (width 1.5) (layer F.Cu) (net 64))
   (segment (start 49 13.5) (end 51.75 13.5) (width 1.5) (layer F.Cu) (net 65))
+  (segment (start 63.737898 86.043949) (end 63.543949 86.043949) (width 0.5) (layer F.Cu) (net 66))
   (zone (net 1) (net_name GND) (layer F.Cu) (hatch edge 0.508)
     (connect_pads (clearance 0.3))
