File: aquarium.kicad_pcb (KiCad board)
At the start: 2 copper layers, 96.2 x 98 mm, 73 parts, among them T1 E16, U1 MOC3063, U2 PC817A

Commit message: README totally reworked.
Parts:
- C10: value 6.8мк -> 6.8u
- C11: value 22мк -> 22u
- C12: value 100н -> 100n
- C13: value 10н -> 10n
- C14: value 2н2 -> 2n2
- C15: value 1000мк -> 1000u
- C16: value 100мк -> 100u
- C17: value 47мк -> 47u
- GB1: value 3В -> 3V
- L1: value 1мГн -> 1mH
- L2: value 100мкГн -> 100uH
- R14: value 1к -> 1k
- R17: value 2к -> 2k
- RU1: value 275B -> 275V
Connections:
- net +12B renamed +12V
- net +5B renamed +5V
