File: aquarium.sch (KiCad schematic (older format))
At the start: 33 parts

Commit message: Schematic/PCB update to the latest KiCad.
Parts:
- C1, C2, C3, C4, C5, C6, C7, C8, C9: symbol C -> Конденсаторы:C
- DD1: symbol ATMEGA8_EXT -> Микроконтроллеры:ATMEGA8_EXT
- DD2, DD3: symbol AT42QT1011 -> Преобразователи:AT42QT1011
- DD4: symbol DS1302 -> Микроконтроллеры:DS1302
- DD5: symbol DS18B20 -> Датчики:DS18B20
- GB1: symbol BAT -> Прочее:BAT
- HG1: symbol CA56-21EWA -> Индикаторы:CA56-21EWA
- R1, R18, R2, R3, R4, R5, R6, R7, R8: symbol R.125 -> Резисторы:R.125
- VT1: symbol IRLD014 -> Транзисторы_полевые:IRLD014
- XP1, XP2: symbol Pin -> Разъемы:Pin
- XT1, XT3: symbol PLS-4 -> Разъемы:PLS-4
- XT2: symbol PLD-6 -> Разъемы:PLD-6
- XT4: symbol 282844-2 -> Разъемы:282844-2
- ZQ1: symbol QUARTZ -> Резонаторы:QUARTZ
