File: power.sch (KiCad schematic (older format))
At the start: 38 parts, among them T1 E16, U1 MOC3063, U2 PC817A

Commit message: Small changes to PCB.
Parts:
- C13: footprint Конденсаторы:C_7.5x4mm -> Конденсаторы:C_5x3mm
Changed lines of the file:
@@
 F 0 "C13" H 11431 3129 138 0000 L CNN
 F 1 "10н" H 11431 2900 138 0000 L CNN
-F 2 "Конденсаторы:C_7.5x4mm" H 11250 2925 60  0001 C CNN
+F 2 "Конденсаторы:C_5x3mm" H 11250 2925 60  0001 C CNN
 F 3 "" H 11250 2925 60  0000 C CNN
 F 4 "1кВ" H 11431 2671 138 0000 L CNN "Тип"

Commit message: README totally reworked.
Parts:
- C10: value 6.8мк -> 6.8u; Тип 400В -> 400V
- C11: value 22мк -> 22u; Тип 400В -> 400V
- C12: value 100н -> 100n; Тип 50В -> 50V
- C13: value 10н -> 10n; Тип 1кВ -> 1kV
- C14: value 2н2 -> 2n2; Тип ~~250В -> ~~250V
- C15: value 1000мк -> 1000u; Тип 25В -> 25V
- C16: value 100мк -> 100u; Тип 25В -> 25V
- C17: value 47мк -> 47u; Тип 35В -> 35V
- L1: value 1мГн -> 1mH
- L2: value 100мкГн -> 100uH
- R11: footprint Резисторы:RV_0.25 -> Резисторы:RH_0.25
- R14: value 1к -> 1k
- R17: value 2к -> 2k
- RU1: value 275B -> 275V
Connections:
- net +12B renamed +12V
- net +5B renamed +5V
Other:
- note added: "+12V"
- note added: "+5V"
- note added: "Core: E16/8/5\nBobbin: EE16-K-H-8P-SS\nI: 215 x 0.15mm\nII: 16 x 0.6mm (12V, 0.5A)"
- note added: "GND"
- note added: "HEAT"
- note added: "HEATER"
- note added: "I"
- note added: "II"
- note added: "T1"
- note added: "~~220V"
- note removed: "+12В"
- note removed: "+5В"
- note removed: "~~220В"
- note removed: "Нагрев."
- note removed: "Общ."
- note removed: "Упр. нагр."
Changed lines of the file:
@@
-EESchema Schematic File Version 2
+EESchema Schematic File Version 3
 LIBS:power
 LIBS:Выключатели_и_кнопки
@@
 	2000 6550 3800 6550
 $Comp
-L GND #PWR25
+L GND #PWR025
 U 1 1 58478AE9
 P 5800 6450
-F 0 "#PWR25" H 6200 6450 138 0001 C CNN
+F 0 "#PWR025" H 6200 6450 138 0001 C CNN
 F 1 "GND" H 5450 6450 138 0001 C CNN
 F 2 "" H 5800 6450 60  0000 C CNN
@@
 F 0 "R11" H 7000 5250 138 0000 C CNN
 F 1 "620" H 7000 4850 138 0000 C CNN
-F 2 "Резисторы:RV_0.25" H 7000 5050 60  0001 C CNN
+F 2 "Резисторы:RH_0.25" H 7000 5050 60  0001 C CNN
 F 3 "" H 7000 5050 60  0000 C CNN
 	1    7000 5050
@@
 $EndComp
 Text Notes 650  3175 0    98   ~ 0
-~~220В
+~~220V
 Text Notes 650  3375 0    98   ~ 0
-~~220В
+~~220V
 Text Notes 650  6425 0    98   ~ 0
-Нагрев.
+HEATER
 Text Notes 650  6625 0    98   ~ 0
-Нагрев.
+HEATER
 Connection ~ 3400 6550
 Connection ~ 3250 5050
 $Comp
-L +5B #PWR30
+L +5V #PWR030
 U 1 1 5847A05B
 P 18600 1850
-F 0 "#PWR30" H 19100 1950 138 0001 C CNN
-F 1 "+5B" H 18584 2285 138 0000 C CNN
+F 0 "#PWR030" H 19100 1950 138 0001 C CNN
+F 1 "+5V" H 18584 2285 138 0000 C CNN
 F 2 "" H 18600 2050 60  0000 C CNN
 F 3 "" H 18600 2050 60  0000 C CNN
@@
 $EndComp
 Text Notes 18975 5075 2    98   ~ 0
-+5В
-Text Notes 19200 5450 2    98   ~ 0
-Упр. нагр.
++5V
+Text Notes 19025 5450 2    98   ~ 0
+HEAT
 Text Notes 19025 4875 2    98   ~ 0
-+12В
++12V
 Text Notes 18975 5275 2    98   ~ 0
-Общ.
+GND
 Text Notes 19150 5750 2    138  ~ 0
 POWER
@@
 P 8750 3200
 F 0 "C11" H 8931 3435 138 0000 L CNN
-F 1 "22мк" H 8931 3206 138 0000 L CNN
+F 1 "22u" H 8931 3206 138 0000 L CNN
 F 2 "Конденсаторы:CPH_5_13x25mm" H 8750 3225 60  0001 C CNN
 F 3 "" H 8750 3225 60  0000 C CNN
-F 4 "400В" H 8931 2977 138 0000 L CNN "Тип"
+F 4 "400V" H 8931 2977 138 0000 L CNN "Тип"
 	1    8750 3200
 	1    0    0    -1
@@
 P 8050 4500
 F 0 "L1" H 8050 4975 138 0000 C CNN
-F 1 "1мГн" H 8050 4746 138 0000 C CNN
+F 1 "1mH" H 8050 4746 138 0000 C CNN
 F 2 "Дроссели:Ind_5x8mm" V 7650 4850 60  0001 C CNN
 F 3 "" V 7650 4850 60  0000 C CNN
@@
 P 3250 3200
 F 0 "RU1" H 3481 3308 138 0000 L CNN
-F 1 "275B" H 3481 3079 138 0000 L CNN
+F 1 "275V" H 3481 3079 138 0000 L CNN
 F 2 "Резисторы:FNR-05" V 3250 3200 60  0001 C CNN
 F 3 "" V 3250 3200 60  0000 C CNN
@@
 P 7350 3200
 F 0 "C10" H 7531 3435 138 0000 L CNN
-F 1 "6.8мк" H 7531 3206 138 0000 L CNN
+F 1 "6.8u" H 7531 3206 138 0000 L CNN
 F 2 "Конденсаторы:CPH_5_10x16mm" H 7350 3225 60  0001 C CNN
 F 3 "" H 7350 3225 60  0000 C CNN
-F 4 "400В" H 7531 2977 138 0000 L CNN "Тип"
+F 4 "400V" H 7531 2977 138 0000 L CNN "Тип"
 	1    7350 3200
 	1    0    0    -1
@@
 P 10400 2900
 F 0 "R14" V 10500 3000 138 0000 L CNN
-F 1 "1к" V 10300 3000 138 0000 L CNN
+F 1 "1k" V 10300 3000 138 0000 L CNN
 F 2 "Резисторы:RV_0.25" H 10400 2900 60  0001 C CNN
 F 3 "" H 10400 2900 60  0000 C CNN
@@
 P 11250 2900
 F 0 "C13" H 11431 3129 138 0000 L CNN
-F 1 "10н" H 11431 2900 138 0000 L CNN
+F 1 "10n" H 11431 2900 138 0000 L CNN
 F 2 "Конденсаторы:C_5x3mm" H 11250 2925 60  0001 C CNN
 F 3 "" H 11250 2925 60  0000 C CNN
-F 4 "1кВ" H 11431 2671 138 0000 L CNN "Тип"
+F 4 "1kV" H 11431 2671 138 0000 L CNN "Тип"
 	1    11250 2900
 	1    0    0    -1
@@
 P 9600 6100
 F 0 "C12" H 9780 6329 138 0000 L CNN
-F 1 "100н" H 9780 6100 138 0000 L CNN
+F 1 "100n" H 9780 6100 138 0000 L CNN
 F 2 "Конденсаторы:C_5x3mm" H 9600 6125 60  0001 C CNN
 F 3 "" H 9600 6125 60  0000 C CNN
-F 4 "50В" H 9780 5871 138 0000 L CNN "Тип"
+F 4 "50V" H 9780 5871 138 0000 L CNN "Тип"
 	1    9600 6100
 	-1   0    0    -1
@@
 P 15050 2450
 F 0 "C15" H 15231 2685 138 0000 L CNN
-F 1 "1000мк" H 15231 2456 138 0000 L CNN
+F 1 "1000u" H 15231 2456 138 0000 L CNN
 F 2 "Конденсаторы:CPH_5_10x20mm" H 15050 2475 60  0001 C CNN
 F 3 "" H 15050 2475 60  0000 C CNN
-F 4 "25В" H 15250 2200 138 0000 L CNN "Тип"
+F 4 "25V" H 15250 2200 138 0000 L CNN "Тип"
 	1    15050 2450
 	1    0    0    -1
@@
 P 17100 2450
 F 0 "C16" H 16900 2700 138 0000 R CNN
-F 1 "100мк" H 16900 2450 138 0000 R CNN
+F 1 "100u" H 16900 2450 138 0000 R CNN
 F 2 "Конденсаторы:CP_2.5x6mm" H 17100 2475 60  0001 C CNN
 F 3 "" H 17100 2475 60  0000 C CNN
-F 4 "25В" H 16900 2200 138 0000 R CNN "Тип"
+F 4 "25V" H 16900 2200 138 0000 R CNN "Тип"
 	1    17100 2450
 	1    0    0    -1
@@
 P 16100 2050
 F 0 "L2" H 16100 2525 138 0000 C CNN
-F 1 "100мкГн" H 16100 2296 138 0000 C CNN
+F 1 "100uH" H 16100 2296 138 0000 C CNN
 F 2 "Дроссели:Ind_5x8mm" V 15700 2400 60  0001 C CNN
 F 3 "" V 15700 2400 60  0000 C CNN
@@
 P 15200 5600
 F 0 "R17" V 15085 5706 138 0000 L CNN
-F 1 "2к" V 15314 5706 138 0000 L CNN
+F 1 "2k" V 15314 5706 138 0000 L CNN
 F 2 "Резисторы:RV_0.25" H 15200 5600 60  0001 C CNN
 F 3 "" H 15200 5600 60  0000 C CNN
@@
 	13000 2050 13600 2050
 $Comp
-L +12B #PWR28
+L +12V #PWR028
 U 1 1 586E9623
 P 17100 1900
-F 0 "#PWR28" H 17600 2000 138 0001 C CNN
-F 1 "+12B" H 17087 2345 138 0000 C CNN
+F 0 "#PWR028" H 17600 2000 138 0001 C CNN
+F 1 "+12V" H 17087 2345 138 0000 C CNN
 F 2 "" H 17100 2100 60  0000 C CNN
 F 3 "" H 17100 2100 60  0000 C CNN
@@
 $EndComp
 $Comp
-L GND #PWR31
+L GND #PWR031
 U 1 1 586E9961
 P 18600 3000
-F 0 "#PWR31" H 19000 3000 138 0001 C CNN
+F 0 "#PWR031" H 19000 3000 138 0001 C CNN
 F 1 "GND" H 18250 3000 138 0001 C CNN
 F 2 "" H 18600 3000 60  0000 C CNN
@@
 P 18600 2450
 F 0 "C17" H 18781 2685 138 0000 L CNN
-F 1 "47мк" H 18781 2456 138 0000 L CNN
+F 1 "47u" H 18781 2456 138 0000 L CNN
 F 2 "Конденсаторы:CP_2.5x5mm" H 18600 2475 60  0001 C CNN
 F 3 "" H 18600 2475 60  0000 C CNN
-F 4 "35В" H 18800 2200 138 0000 L CNN "Тип"
+F 4 "35V" H 18800 2200 138 0000 L CNN "Тип"
 	1    18600 2450
 	1    0    0    -1
@@
 	17500 5400 17700 5400
 $Comp
-L GND #PWR27
+L GND #PWR027
 U 1 1 586EFA44
 P 16800 5350
-F 0 "#PWR27" H 17200 5350 138 0001 C CNN
+F 0 "#PWR027" H 17200 5350 138 0001 C CNN
 F 1 "GND" H 16450 5350 138 0001 C CNN
 F 2 "" H 16800 5350 60  0000 C CNN
@@
 	16800 5200 17700 5200
 $Comp
-L +12B #PWR29
+L +12V #PWR029
 U 1 1 586EFC16
 P 17500 4400
-F 0 "#PWR29" H 18000 4500 138 0001 C CNN
-F 1 "+12B" H 17487 4845 138 0000 C CNN
+F 0 "#PWR029" H 18000 4500 138 0001 C CNN
+F 1 "+12V" H 17487 4845 138 0000 C CNN
 F 2 "" H 17500 4600 60  0000 C CNN
 F 3 "" H 17500 4600 60  0000 C CNN
@@
 $EndComp
 $Comp
-L +5B #PWR26
+L +5V #PWR026
 U 1 1 586EFC90
 P 16800 4400
-F 0 "#PWR26" H 17300 4500 138 0001 C CNN
-F 1 "+5B" H 16784 4835 138 0000 C CNN
+F 0 "#PWR026" H 17300 4500 138 0001 C CNN
+F 1 "+5V" H 16784 4835 138 0000 C CNN
 F 2 "" H 16800 4600 60  0000 C CNN
 F 3 "" H 16800 4600 60  0000 C CNN
@@
 P 12550 1150
 F 0 "C14" V 11769 1150 138 0000 C CNN
-F 1 "2н2" V 11998 1150 138 0000 C CNN
+F 1 "2n2" V 11998 1150 138 0000 C CNN
 F 2 "Конденсаторы:C_7.5x4mm" H 12550 1175 60  0001 C CNN
 F 3 "" H 12550 1175 60  0000 C CNN
-F 4 "~~250В" V 12241 1150 138 0000 C CNN "Тип"
+F 4 "~~250V" V 12241 1150 138 0000 C CNN "Тип"
 	1    12550 1150
 	0    1    1    0
@@
 	13250 1150 13250 2850
 Connection ~ 13250 2850
+Text Notes 12225 2550 0    138  ~ 0
+I
+Text Notes 12900 2550 0    138  ~ 0
+II
+Text Notes 1850 800  0    138  ~ 28
+T1
+Text Notes 925  1775 0    138  ~ 0
+Core: E16/8/5\nBobbin: EE16-K-H-8P-SS\nI: 215 x 0.15mm\nII: 16 x 0.6mm (12V, 0.5A)
 $EndSCHEMATC

Commit message: Schematic/PCB update to the latest KiCad.
Parts:
- C10, C11, C15, C16, C17: symbol Cpol -> Конденсаторы:Cpol
- C12, C13, C14: symbol C -> Конденсаторы:C
- DA1: symbol TNY274 -> Преобразователи:TNY274
- DA2: symbol 78L05 -> Стабилизаторы:78L05
- FU1: symbol Fuse -> Предохранители:Fuse
- L1, L2: symbol Coil -> Дроссели:Coil
- R10, R9: symbol R2 -> Резисторы:R2
- R11: symbol R.125 -> Резисторы:R.125
- R12, R13, R14, R15, R16, R17: symbol R.25 -> Резисторы:R.25
- RU1: symbol R_U_vert -> Резисторы:R_U_vert
- T1: symbol E16 -> Трансформаторы:E16
- U1: symbol MOC3063 -> Оптопары:MOC3063
- U2: symbol PC817 -> Оптопары:PC817
- VD1, VD2, VD3, VD4, VD6: symbol 1N4007 -> Диоды:1N4007
- VD5, VD8: symbol Zener -> Диоды:Zener
- VD7: symbol Schottky -> Диоды:Schottky
- VS1: symbol BT137 -> Тиристоры:BT137
- XT5, XT6: symbol 282844-2 -> Разъемы:282844-2
- XT7: symbol PLS-4 -> Разъемы:PLS-4
